Commit message: ajustado caminho absoluto

File: src/manipulator_description_pkg/urdf/manipulator_description_gazebo.urdf (robot description, URDF)
Before this commit: robot manipulator_description, 9 links, 8 joints
Links:
- link Link_1: geometry collision mesh filename=package://manipulator_description_pkg/meshes/Link_1.stl; visual mesh filename=package://manipulator_description_pkg/meshes/Link_1.stl
- link Link_2: geometry collision mesh filename=package://manipulator_description_pkg/meshes/Link_2.stl; visual mesh filename=package://manipulator_description_pkg/meshes/Link_2.stl
- link Link_3: geometry collision mesh filename=package://manipulator_description_pkg/meshes/Link_3.stl; visual mesh filename=package://manipulator_description_pkg/meshes/Link_3.stl
- link Link_4: geometry collision mesh filename=package://manipulator_description_pkg/meshes/Link_4.stl; visual mesh filename=package://manipulator_description_pkg/meshes/Link_4.stl
- link Link_5: geometry collision mesh filename=package://manipulator_description_pkg/meshes/Link_5.stl; visual mesh filename=package://manipulator_description_pkg/meshes/Link_5.stl
- link Link_6: geometry collision mesh filename=package://manipulator_description_pkg/meshes/Link_6.stl; visual mesh filename=package://manipulator_description_pkg/meshes/Link_6.stl
- link Link_7: geometry collision mesh filename=package://manipulator_description_pkg/meshes/Link_7.stl; visual mesh filename=package://manipulator_description_pkg/meshes/Link_7.stl
- link base_link: geometry collision mesh filename=package://manipulator_description_pkg/meshes/base_link.stl; visual mesh filename=package://manipulator_description_pkg/meshes/base_link.stl
